Commit message: actualizacion1

File: urdf/omnibot2.urdf (robot description, URDF)
Before this commit: robot robot, 4 links, 3 joints
Links:
- added link leftback_link, mass 0.1; collision cylinder length=0.05 radius=0.05; visual mesh filename=package://ign_robots_examples/meshes/right_mecanum_wheel.dae scale=1.0 0.8 1.0
- added link leftfront_link, mass 0.1; collision cylinder length=0.05 radius=0.05; visual mesh filename=package://ign_robots_examples/meshes/left_mecanum_wheel.dae scale=1.0 0.8 1.0
- added link rightback_link, mass 0.1; collision cylinder length=0.05 radius=0.05; visual mesh filename=package://ign_robots_examples/meshes/left_mecanum_wheel.dae scale=1.0 0.8 1.0
- added link rightfront_link, mass 0.1; collision cylinder length=0.05 radius=0.05; visual mesh filename=package://ign_robots_examples/meshes/right_mecanum_wheel.dae scale=1.0 0.8 1.0
Joints:
- added joint leftback_joint: type continuous, parent base_link, child leftback_link, origin xyz=-0.085 0.14 0.01 rpy=-1.570796325 0 0, axis 0 0 1
- added joint leftfront_joint: type continuous, parent base_link, child leftfront_link, origin xyz=0.085 0.14 0.01 rpy=-1.570796325 0 0, axis 0 0 1
- added joint rightback_joint: type continuous, parent base_link, child rightback_link, origin xyz=-0.085 -0.14 0.01 rpy=-1.570796325 0 0, axis 0 0 1
- added joint rightfront_joint: type continuous, parent base_link, child rightfront_link, origin xyz=0.085 -0.14 0.01 rpy=-1.570796325 0 0, axis 0 0 1
- joint base_joint: origin xyz=0 0 ${base_elevation} rpy=0 0 0 -> xyz=0 0 0.08 rpy=0 0 0
